File: boards/esp32s3-devkit-5v/esp32s3-devkit-5v.kicad_sch (KiCad schematic)
At the start: 81 parts, among them J1 Conn_01x02_Pin, J2 USB_C_Receptacle_USB2.0_16P, J3 Conn_01x02_Pin, J4 Conn_01x04_Pin, Q1 AO3401A, Q2 AO3401A, Q3 MMBT3904, SW1 MK-12C03-G015, SW2 RESET, SW3 BOOT, SW4 SW_Push, SW5 SW_Push, SW6 SW_Push, SW7 SW_Push, U1 TPS63070RNMR, U2 TPS63070RNMR, U3 ESP32-S3-WROOM-1-N16, U4 USBLC6-2SC6, U5 RV-3028-C7, U6 MAX98357A

Commit message: feat(esp32s3-devkit-5v): add compact dual-rail PCB and physical screening (#122)
* feat(esp32s3-devkit-5v): add reviewed schematic and routed prototype

* Compact dual-rail PCB and add safe power monitoring

* fix(pcb): restore close converter bypass placement and guard it

* test(pcb): add physical screening and compact-layout test report

* fix(ci): build FastHenry with portable scalar compiler settings

* fix(ci): rebuild cached FastHenry objects with selected flags

* fix(sim): repair FastHenry sparse statistics adapter pointer

* test(pcb): model three-AA power limits and define bench validation

* test(audio): screen continuous alarm loads and document speaker proposal

* docs(audio): define bedroom wake-up validation and refresh evidence
Parts:
- added C29, C30, C32, C33: 0.1µF, Capacitor_SMD:C_0402_1005Metric, symbol Device:C
- added C31: 1µF, Capacitor_SMD:C_0603_1608Metric, symbol Device:C
- added R31, R33: 10kΩ, Resistor_SMD:R_0402_1005Metric, symbol Device:R
- added R32, R36, R39: 100kΩ, Resistor_SMD:R_0402_1005Metric, symbol Device:R
- added R34, R35: 22Ω, Resistor_SMD:R_0402_1005Metric, symbol Device:R
- added R37, R38: 4.7kΩ, Resistor_SMD:R_0402_1005Metric, symbol Device:R
- added U7: SN74LVC2G66DCUR, Package_SO:VSSOP-8_2.3x2mm_P0.5mm, symbol Review:SN74LVC2G66DCUR
- added U8: SN74LVC1T45DBVR, Package_TO_SOT_SMD:SOT-23-6, symbol Review:SN74LVC1T45DBVR
- C1, C10, C12, C17, C18, C19, C2, C20, C21, C22, C23, C24, C25, C26, C27, C28, C4, C9: Dielectric (none) -> X5R or X7R; Voltage (none) -> 10V minimum
- C11, C13, C3, C5: footprint Capacitor_SMD:C_0402_1005Metric -> Capacitor_SMD:C_0603_1608Metric; Dielectric (none) -> X5R or X7R; Voltage (none) -> 10V minimum
- C14, C15, C16, C6, C7, C8: footprint Capacitor_SMD:C_0805_2012Metric -> Capacitor_SMD:C_1206_3216Metric; Dielectric (none) -> X5R or X7R; MPN (none) -> GRM31CR61C226KE15L; Voltage (none) -> 16V
- D2: renamed from D4; value LED_RGBK -> 150141M173100; symbol Device:LED_RGBK -> Review:WE_150141M173100; MPN (none) -> 150141M173100
- J2: footprint Connector_USB:USB_C_Receptacle_HRO_TYPE-C-31-M-12 -> Board:USB_C_HRO_Overhang
- J3: footprint Connector_JST:JST_PH_B2B-PH-SM4-TB_1x02-1MP_P2.00mm_Vertical -> Board:JST_PH_Speaker_Overhang
- L1, L2: MPN (none) -> XFL4020-152MEC
- R11: Assembly note (none) -> DNP for battery operation; fit for power indicator; now not fitted
- R14, R15, R4, R5, R8, R9: Tolerance (none) -> 1%
- SW1: value MK-12C03-G015 -> MSK12C02; MPN (none) -> MSK12C02
- SW4: value SW_Push -> VOL-
- SW5: value SW_Push -> MODE
- SW6: value SW_Push -> VOL+
- SW7: value SW_Push -> BATTERY
- U3: footprint RF_Module:ESP32-S3-WROOM-1 -> Board:ESP32-S3-WROOM-1_Overhang
- renumbered D3 to D1
Connections:
- net 3v3: now also D2.1 (A), R10.1, C29.1, C30.1, C32.1, U7.8 (VCC), U8.1 (VCCA), U8.5 (DIR); no longer U5.6 (VBACKUP)
- net 5v: now also C33.1, U8.6 (VCCB); no longer R10.1
- net D+: now also R35.2; no longer U3.14 (USB_D+)
- net D-: now also R34.2; no longer U3.13 (USB_D-)
- net GND: now also SW1.3 (C), C29.2, C30.2, C31.2, C32.2, C33.2, R32.2, R33.2, R36.2, R39.2, U7.4 (GND), U8.2 (GND); no longer D2.4 (K)
- net GPIO15: now also R6.2, U1.2 (PG); no longer U6.16 (BCLK)
- net GPIO21: now also R39.1, U8.3 (A); no longer R20.1, U6.4 (~{SD_MODE})
- net GPIO7: no longer R22.2
- net GPIO8: now also U7.5 (2A); no longer J4.4 (Pin_4)
- net GPIO9: now also U7.1 (1A); no longer J4.3 (Pin_3)
- net PFET: now also C1.1, C10.1, C11.1, C2.1, C3.1, C9.1, R3.1, R7.1, U1.12 (VIN), U1.13 (VIN), U2.12 (VIN), U2.13 (VIN), R31.1; no longer SW1.2 (B)
- net GPIO11: now reaches U3.19 (IO11)
- net GPIO11: now also R36.1, U7.3 (2C), U7.7 (1C)
- net GPIO12: now reaches U3.20 (IO12)
- net GPIO13: now reaches U3.21 (IO13)
- net GPIO13: now also R10.2, U2.2 (PG)
- net GPIO14: now reaches U3.22 (IO14)
- net GPIO14: now also U6.1 (DIN)
- net GPIO47: now reaches U3.24 (IO47)
- net GPIO47: now also U6.16 (BCLK)
- net GPIO48: now reaches U3.25 (IO48)
- net GPIO48: now also U6.14 (LRCLK)
- net GPIO41: now reaches U3.34 (IO41)
- net GPIO41: now also R22.2
- net GPIO2: now reaches U3.38 (IO2)
- net at R30.1: now also D2.2 (BK); no longer D2.3 (BA)
- net USB_VBUS: now reaches C20.1, J2.A4 (VBUS), J2.A9 (VBUS), J2.B4 (VBUS), J2.B9 (VBUS), U4.5 (VBUS)
- net USB_VBUS: no longer J2.A5 (CC1), R15.1
- net at R3.2, U1.1 (PS_SYNC): no longer U1.14 (EN)
- net at R29.1: now also D2.4 (GK); no longer D2.2 (GA)
- net at R28.1: now also D2.3 (RK); no longer D2.1 (RA)
- net GPIO16: no longer names the net of U3.9 (IO16)
- net GPIO16: no longer U6.14 (LRCLK)
- net GPIO17: no longer names the net of U3.10 (IO17)
- net GPIO17: no longer U6.1 (DIN)
- removed net VBAT_SW: C1.1, C10.1, C11.1, C2.1, C3.1, C9.1, R3.1, R7.1, SW1.1 (A), U1.12 (VIN), U1.13 (VIN), U2.12 (VIN), U2.13 (VIN)
- net VCC renamed OLED_3V3
- net OLED_3V3: now also C31.1, R37.1, R38.1
- new net AMP_SD: R20.1, U6.4 (~{SD_MODE}), U8.4 (B)
- new net EN_3V3: R32.1, SW1.2 (B), U1.14 (EN)
- new net OLED_SCL: J4.3 (Pin_3), R37.2, U7.2 (1B)
- new net OLED_SDA: J4.4 (Pin_4), R38.2, U7.6 (2B)
- new net RTC_VBACKUP: R33.1, U5.6 (VBACKUP)
- new net SW_ON: R31.2, SW1.1 (A)
- new net USB_CC1: J2.A5 (CC1), R15.1
- new net USB_MCU_N: R34.1, U3.13 (USB_D-)
- new net USB_MCU_P: R35.1, U3.14 (USB_D+)
- no-connect marks 21 -> 14
Other:
- added sheet Power monitoring (power-monitor.kicad_sch)
- note added: "D2: common anode at 3V3; RGB GPIO LOW = ON. Wuerth 150141M173100: A=1, R=3, G=4, B=2."
- note added: "DESIGN REVIEW 2026-09-04 | Prototype; battery/load and enclosure pending confirmation. TPS63070: PS/SYNC HIGH = power save (both rails). 3.31V / 4.985V nominal. Cold start requires >=3.0V at converter input. JST-PH input rated 2A with specified wire. USB is data-only: VBUS supplies ESD bias only. R11 DNP for low standby current. RTC backup/trickle charge OFF; time is lost when main power is off. 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"
- note added: "OLED: GPIO41 = power, GPIO11 = bus connect (both default OFF). ON: GPIO41 high, wait for supply, GPIO11 high. OFF: GPIO11 low, then GPIO41 low. J4 order: GND / switched 3V3 / SCL / SDA. Verify display pinout."
- note added: "Routing GPIO map: BCLK=47, LRCLK=48, DIN=14; OLED power=41. Other assigned GPIOs retained; firmware changes in review/gpio-map.csv."
- note added: "SW1 selects EN_3V3: ON = PFET via R31; OFF = GND. Battery current bypasses SW1; this is standby, not battery isolation."
- note removed: "0402 X5R"
- note removed: "0402 X7R"
- note removed: "0805 X6S"
- note removed: "0805 X7S"
- moved on the sheet: R10, SW1
