File: boards/alec-sensor/alec-sensor.kicad_pcb (KiCad board)
At the start: 4 copper layers, 64 x 56 mm, 100 parts, among them J1 Conn_01x02_Pin, J2 USB_C_Receptacle_USB2.0_16P, J3 LD2410C — INTERNAL, Q1 AO3401A, Q4 MMBT3904, Q5 MMBT3904, Q6 AO3401A, Q7 MMBT3904, SW1 1101M2S3CQE2, SW2 RESET, SW3 BOOT, SW7 BATTERY / PAIR, U1 TPS63070RNMR, U10 TMUX1511PWR, U2 TPS63070RNMR, U3 ESP32-S3-WROOM-1-N16, U4 USBLC6-2SC6, U5 RV-3028-C7

Commit message: fix: expose ALEC Sensor batteries and controls through rear cover
Parts:
- SW2, SW3: moved to B.Cu
- moved SW3 41.3 mm to (130.0, 85.0), turned to 180 degrees
- moved SW2 11.4 mm to (115.0, 85.0), turned to 180 degrees
- moved SW1 3.00 mm to (153.0, 86.5)
Routing:
- net Net-(U3-IO0): track 47.3 -> 22.7 mm, vias 4 -> 5
- net /RADAR_TX: track 33.5 -> 50.8 mm, vias 5 -> 6
- net /3v3: track 196.5 -> 211.1 mm, vias 13 -> 14
- net GND: track 94.1 -> 107.4 mm, vias 77 -> 79
- net Net-(U3-EN): track 17.7 -> 26.7 mm, vias 2 -> 3
- net /GPIO9: track 35.4 -> 39.2 mm, vias 4 -> 3
- net /VBAT_FUSED: track 52.0 -> 55.1 mm
- net /RADAR_EN: track 41.8 -> 44.2 mm
- net /VBAT_SW: track 53.4 -> 54.3 mm
Other:
- board text added: "ALEC SENSOR S1.1"
- board text added: "RESET"
- board text removed: "ALEC SENSOR S1"
