File: boards/alec-sensor/alec-sensor.kicad_sch (KiCad schematic)
At the start: 65 parts, among them J1 Conn_01x02_Pin, J2 USB_C_Receptacle_USB2.0_16P, Q1 AO3401A, SW1 1101M2S3CQE2, SW2 RESET, SW3 BOOT, SW7 BATTERY / PAIR, U1 TPS63070RNMR, U2 TPS63070RNMR, U3 ESP32-S3-WROOM-1-N16, U4 USBLC6-2SC6, U5 RV-3028-C7

Commit message: fix: align sensor capacitor BOM and plan paired prototype order
Parts:
- C29: MPN GRM188R71C104KA01D -> GRM155R71C104KA88D
Changed lines of the file:
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@@
 		(property
 			"Datasheet"
-			"https://www.murata.com/en-us/products/productdetail?partno=GRM188R71C104KA01D"
+			"https://search.murata.co.jp/Ceramy/image/img/A01X/G101/ENG/GRM155R71C104KA88-01A.pdf"
 			(at 251.4600 125.7300 0)
 			(hide yes)
@@
 		(property
 			"MPN"
-			"GRM188R71C104KA01D"
+			"GRM155R71C104KA88D"
 			(at 0 0 0)
 			(effects
